Commit message: (experimental) modifications according to ur macro xacro

File: urdf/kuka_macro.xacro (robot description, xacro)
@@ -259,4 +259,21 @@
         velocity="${joint_6_velocity_limit}" />
     </joint>
+    <link name="${tf_prefix}ft_frame"/>
+    <joint name="${tf_prefix}link_6-ft_frame" type="fixed">
+      <parent link="${tf_prefix}link_6"/>
+      <child link="${tf_prefix}ft_frame"/>
+      <origin xyz="0 0 0" rpy="${pi} 0 0"/>
+    </joint>
+    <link name="${tf_prefix}base"/>
+    <joint name="${tf_prefix}base_link-base_fixed_joint" type="fixed">
+      <!-- Note the rotation over Z of pi radians - as base_link is REP-103
+           aligned (i.e., has X+ forward, Y+ left and Z+ up), this is needed
+           to correctly align 'base' with the 'Base' coordinate system of
+           the UR controller.
+      -->
+      <origin xyz="0 0 0" rpy="0 0 ${pi}"/>
+      <parent link="${tf_prefix}base_link"/>
+      <child link="${tf_prefix}base"/>
+    </joint>
     <!-- ROS-Industrial 'flange' frame - attachment point for EEF models -->
     <link name="${tf_prefix}flange" />

Commit message: fix robot model tf

File: urdf/kuka_macro.xacro (robot description, xacro)
@@ -52,6 +52,5 @@
       force_abs_paths="${force_abs_paths}" />
     <!-- Links -main serial chain -->
-    <link name="${tf_prefix}base_link" />
-    <link name="${tf_prefix}base_link_inertia">
+    <link name="${tf_prefix}base_link">
       <visual>
         <origin xyz="0 0 0" rpy="0 0 0" />
@@ -187,19 +186,13 @@
     </link>
     <!-- base_joint fixes base_link to the environment -->
-    <joint name="${tf_prefix}base_joint" type="fixed">
+    <joint name="${tf_prefix}${parent}-base_link" type="fixed">
       <parent link="${parent}" />
       <child link="${tf_prefix}base_link" />
       <xacro:insert_block name="origin" />
     </joint>
-    <!-- ROS base_link to KUKA $ROBROOT coordinate system transform -->
-    <joint name="${tf_prefix}base_link-base_link_inertia" type="fixed">
-      <parent link="${tf_prefix}base_link" />
-      <child link="${tf_prefix}base_link_inertia" />
-      <origin xyz="0 0 0" rpy="0 0 0" />
-    </joint>
     <!-- joints - main serial chain -->
     <!-- Joint-1 -->
     <joint name="${tf_prefix}joint_1" type="revolute">
-      <parent link="${tf_prefix}base_link_inertia" />
+      <parent link="${tf_prefix}base_link" />
       <child link="${tf_prefix}link_1" />
       <origin xyz="${link1_x} ${link1_y} ${link1_z}" rpy="${link1_roll} ${link1_pitch} ${link1_yaw}" />
@@ -234,5 +227,5 @@
       <child link="${tf_prefix}link_4" />
       <origin xyz="${link4_x} ${link4_y} ${link4_z}" rpy="${link4_roll} ${link4_pitch} ${link4_yaw}" />
-      <axis xyz="0 1 0" />
+      <axis xyz="-1 0 0" />
       <limit lower="${joint_4_lower_limit}" upper="${joint_4_upper_limit}"
         effort="${joint_4_effort_limit}"
@@ -254,29 +247,19 @@
       <child link="${tf_prefix}link_6" />
       <origin xyz="${link6_x} ${link6_y} ${link6_z}" rpy="${link6_roll} ${link6_pitch} ${link6_yaw}" />
-      <axis xyz="0 1 0" />
+      <axis xyz="-1 0 0" />
       <limit lower="${joint_6_lower_limit}" upper="${joint_6_upper_limit}"
         effort="${joint_6_effort_limit}"
         velocity="${joint_6_velocity_limit}" />
     </joint>
-    <link name="${tf_prefix}ft_frame"/>
-    <joint name="${tf_prefix}link_6-ft_frame" type="fixed">
-      <parent link="${tf_prefix}link_6"/>
-      <child link="${tf_prefix}ft_frame"/>
-      <origin xyz="0 0 0" rpy="${pi} 0 0"/>
-    </joint>
-    <link name="${tf_prefix}base"/>
-    <joint name="${tf_prefix}base_link-base_fixed_joint" type="fixed">
-      <!-- Note the rotation over Z of pi radians - as base_link is REP-103
-           aligned (i.e., has X+ forward, Y+ left and Z+ up), this is needed
-           to correctly align 'base' with the 'Base' coordinate system of
-           the UR controller.
-      -->
-      <origin xyz="0 0 0" rpy="0 0 ${pi}"/>
-      <parent link="${tf_prefix}base_link"/>
-      <child link="${tf_prefix}base"/>
+    <!-- ROS base_link to KUKA $ROBROOT coordinate system transform -->
+    <link name="${tf_prefix}base" />
+    <joint name="${tf_prefix}base_link-base" type="fixed">
+      <origin xyz="0 0 0" rpy="0 0 0" />
+      <parent link="${tf_prefix}base_link" />
+      <child link="${tf_prefix}base" />
     </joint>
     <!-- ROS-Industrial 'flange' frame - attachment point for EEF models -->
     <link name="${tf_prefix}flange" />
-    <joint name="${tf_prefix}flange-joint_6" type="fixed">
+    <joint name="${tf_prefix}joint_6-flange" type="fixed">
       <parent link="${tf_prefix}link_6" />
       <child link="${tf_prefix}flange" />

Commit message: Update kinematics configuration and joint axes from config file

File: urdf/kuka_macro.xacro (robot description, xacro)
@@ -196,5 +196,5 @@
       <child link="${tf_prefix}link_1" />
       <origin xyz="${link1_x} ${link1_y} ${link1_z}" rpy="${link1_roll} ${link1_pitch} ${link1_yaw}" />
-      <axis xyz="0 0 -1" />
+      <axis xyz= "${link1_axis}"/>
       <limit lower="${joint_1_lower_limit}" upper="${joint_1_upper_limit}"
         effort="${joint_1_effort_limit}"
@@ -206,5 +206,5 @@
       <child link="${tf_prefix}link_2" />
       <origin xyz="${link2_x} ${link2_y} ${link2_z}" rpy="${link2_roll} ${link2_pitch} ${link2_yaw}" />
-      <axis xyz="0 1 0" />
+      <axis xyz="${link2_axis}"/>
       <limit lower="${joint_2_lower_limit}" upper="${joint_2_upper_limit}"
         effort="${joint_2_effort_limit}"
@@ -216,5 +216,5 @@
       <child link="${tf_prefix}link_3" />
       <origin xyz="${link3_x} ${link3_y} ${link3_z}" rpy="${link3_roll} ${link3_pitch} ${link3_yaw}" />
-      <axis xyz="0 1 0" />
+      <axis xyz="${link3_axis}" />
       <limit lower="${joint_3_lower_limit}" upper="${joint_3_upper_limit}"
         effort="${joint_3_effort_limit}"
@@ -226,5 +226,5 @@
       <child link="${tf_prefix}link_4" />
       <origin xyz="${link4_x} ${link4_y} ${link4_z}" rpy="${link4_roll} ${link4_pitch} ${link4_yaw}" />
-      <axis xyz="-1 0 0" />
+      <axis xyz="${link4_axis}" />
       <limit lower="${joint_4_lower_limit}" upper="${joint_4_upper_limit}"
         effort="${joint_4_effort_limit}"
@@ -236,5 +236,5 @@
       <child link="${tf_prefix}link_5" />
       <origin xyz="${link5_x} ${link5_y} ${link5_z}" rpy="${link5_roll} ${link5_pitch} ${link5_yaw}" />
-      <axis xyz="0 1 0" />
+      <axis xyz="${link5_axis}" />
       <limit lower="${joint_5_lower_limit}" upper="${joint_5_upper_limit}"
         effort="${joint_5_effort_limit}"
@@ -246,5 +246,5 @@
       <child link="${tf_prefix}link_6" />
       <origin xyz="${link6_x} ${link6_y} ${link6_z}" rpy="${link6_roll} ${link6_pitch} ${link6_yaw}" />
-      <axis xyz="-1 0 0" />
+      <axis xyz="${link6_axis}" />
       <limit lower="${joint_6_lower_limit}" upper="${joint_6_upper_limit}"
         effort="${joint_6_effort_limit}"
