Commit message: Add get_material and get_material_values macros

File: urdf/inc/kuka_common.xacro (robot description, xacro)
@@ -33,4 +33,15 @@
     <xacro:get_mesh_path/>
     <mesh filename="${mesh}"/>
+  </xacro:macro>
+  <xacro:macro name="get_material_values" params="name:=^ type:=^">
+    <xacro:get_visual_params />
+    <xacro:property name="material" value="${visual_params['material']['name']}" scope="parent"/>
+    <xacro:property name="color" value="${visual_params['material']['color']}" scope="parent"/>
+  </xacro:macro>
+  <xacro:macro name="get_material" params="name type">
+    <xacro:get_material_values/>
+    <material name="${material}">
+      <color rgba="${color}"/>
+    </material>
   </xacro:macro>
   <xacro:macro name="read_model_data" params="joint_limits_parameters_file kinematics_parameters_file physical_parameters_file visual_parameters_file force_abs_paths">
