Commit message: Add configuration files for KR10 R1100-2 robot

File: urdf/kuka_macro.xacro (robot description, xacro)
@@ -65,8 +65,8 @@
         </geometry>
       </collision>
-      <xacro:cylinder_inertial radius="${base_inertia_radius}" length="${base_inertia_length}"
-        mass="${base_link_mass}">
-        <origin xyz="0 0 0" rpy="0 0 0" />
-      </xacro:cylinder_inertial>
+      <xacro:inertial_block mass="${base_link_mass}" ixx="${base_ixx}" iyy="${base_iyy}"
+        izz="${base_izz}">
+        <origin xyz="0 0 0" rpy="0 0 0" />
+      </xacro:inertial_block>
     </link>
     <!-- Link-1 -->
@@ -84,8 +84,8 @@
         </geometry>
       </collision>
-      <xacro:cylinder_inertial radius="${link_1_inertia_radius}" length="${link_1_inertia_length}"
-        mass="${link_1_mass}">
-        <origin xyz="0 0 0" rpy="0 0 0" />
-      </xacro:cylinder_inertial>
+      <xacro:inertial_block mass="${link_1_mass}" ixx="${link_1_ixx}" iyy="${link_1_iyy}"
+        izz="${link_1_izz}">
+        <origin xyz="0 0 0" rpy="0 0 0" />
+      </xacro:inertial_block>
     </link>
     <!-- Link-2 -->
@@ -103,8 +103,8 @@
         </geometry>
       </collision>
-      <xacro:cylinder_inertial radius="${link_2_inertia_radius}" length="${link_2_inertia_length}"
-        mass="${link_2_mass}">
-        <origin xyz="0 0 0" rpy="0 0 0" />
-      </xacro:cylinder_inertial>
+      <xacro:inertial_block mass="${link_2_mass}" ixx="${link_2_ixx}" iyy="${link_2_iyy}"
+        izz="${link_2_izz}">
+        <origin xyz="0 0 0" rpy="0 0 0" />
+      </xacro:inertial_block>
     </link>
     <!-- Link-3 -->
@@ -122,8 +122,8 @@
         </geometry>
       </collision>
-      <xacro:cylinder_inertial radius="${link_3_inertia_radius}" length="${link_3_inertia_length}"
-        mass="${link_3_mass}">
-        <origin xyz="0 0 0" rpy="0 0 0" />
-      </xacro:cylinder_inertial>
+      <xacro:inertial_block mass="${link_3_mass}" ixx="${link_3_ixx}" iyy="${link_3_iyy}"
+        izz="${link_3_izz}">
+        <origin xyz="0 0 0" rpy="0 0 0" />
+      </xacro:inertial_block>
     </link>
     <!-- Link-4 -->
@@ -141,8 +141,8 @@
         </geometry>
       </collision>
-      <xacro:cylinder_inertial radius="${link_4_inertia_radius}" length="${link_4_inertia_length}"
-        mass="${link_4_mass}">
-        <origin xyz="0 0 0" rpy="0 0 0" />
-      </xacro:cylinder_inertial>
+      <xacro:inertial_block mass="${link_4_mass}" ixx="${link_4_ixx}" iyy="${link_4_iyy}"
+        izz="${link_4_izz}">
+        <origin xyz="0 0 0" rpy="0 0 0" />
+      </xacro:inertial_block>
     </link>
     <!-- Link-5 -->
@@ -160,8 +160,8 @@
         </geometry>
       </collision>
-      <xacro:cylinder_inertial radius="${link_5_inertia_radius}" length="${link_5_inertia_length}"
-        mass="${link_5_mass}">
-        <origin xyz="0 0 0" rpy="0 0 0" />
-      </xacro:cylinder_inertial>
+      <xacro:inertial_block mass="${link_5_mass}" ixx="${link_5_ixx}" iyy="${link_5_iyy}"
+        izz="${link_5_izz}">
+        <origin xyz="0 0 0" rpy="0 0 0" />
+      </xacro:inertial_block>
     </link>
     <!-- Link-6 -->
@@ -179,8 +179,8 @@
         </geometry>
       </collision>
-      <xacro:cylinder_inertial radius="${link_6_inertia_radius}" length="${link_6_inertia_length}"
-        mass="${link_6_mass}">
-        <origin xyz="0 0 0" rpy="0 0 0" />
-      </xacro:cylinder_inertial>
+      <xacro:inertial_block mass="${link_6_mass}" ixx="${link_6_ixx}" iyy="${link_6_iyy}"
+        izz="${link_6_izz}">
+        <origin xyz="0 0 0" rpy="0 0 0" />
+      </xacro:inertial_block>
     </link>
     <!-- base_joint fixes base_link to the environment -->

Commit message: Add link axis properties to kuka_common.xacro

File: urdf/inc/kuka_common.xacro (robot description, xacro)
@@ -145,4 +145,5 @@
     <xacro:property name="link1_pitch" value="${sec_kinematics['link_1']['pitch']}" scope="parent" />
     <xacro:property name="link1_yaw" value="${sec_kinematics['link_1']['yaw']}" scope="parent" />
+    <xacro:property name="link1_axis" value="${sec_kinematics['link_1']['axis']}" scope="parent" />
     <!-- Link 2 -->
     <xacro:property name="link2_x" value="${sec_kinematics['link_2']['x']}" scope="parent" />
@@ -152,4 +153,5 @@
     <xacro:property name="link2_pitch" value="${sec_kinematics['link_2']['pitch']}" scope="parent" />
     <xacro:property name="link2_yaw" value="${sec_kinematics['link_2']['yaw']}" scope="parent" />
+    <xacro:property name="link2_axis" value="${sec_kinematics['link_2']['axis']}" scope="parent" />
     <!-- Link 3 -->
     <xacro:property name="link3_x" value="${sec_kinematics['link_3']['x']}" scope="parent" />
@@ -159,4 +161,5 @@
     <xacro:property name="link3_pitch" value="${sec_kinematics['link_3']['pitch']}" scope="parent" />
     <xacro:property name="link3_yaw" value="${sec_kinematics['link_3']['yaw']}" scope="parent" />
+    <xacro:property name="link3_axis" value="${sec_kinematics['link_3']['axis']}" scope="parent" />
     <!-- Link 4 -->
     <xacro:property name="link4_x" value="${sec_kinematics['link_4']['x']}" scope="parent" />
@@ -166,4 +169,5 @@
     <xacro:property name="link4_pitch" value="${sec_kinematics['link_4']['pitch']}" scope="parent" />
     <xacro:property name="link4_yaw" value="${sec_kinematics['link_4']['yaw']}" scope="parent" />
+    <xacro:property name="link4_axis" value="${sec_kinematics['link_4']['axis']}" scope="parent" />
     <!-- Link 5 -->
     <xacro:property name="link5_x" value="${sec_kinematics['link_5']['x']}" scope="parent" />
@@ -173,4 +177,5 @@
     <xacro:property name="link5_pitch" value="${sec_kinematics['link_5']['pitch']}" scope="parent" />
     <xacro:property name="link5_yaw" value="${sec_kinematics['link_5']['yaw']}" scope="parent" />
+    <xacro:property name="link5_axis" value="${sec_kinematics['link_5']['axis']}" scope="parent" />
     <!-- Link 6 -->
     <xacro:property name="link6_x" value="${sec_kinematics['link_6']['x']}" scope="parent" />
@@ -180,4 +185,5 @@
     <xacro:property name="link6_pitch" value="${sec_kinematics['link_6']['pitch']}" scope="parent" />
     <xacro:property name="link6_yaw" value="${sec_kinematics['link_6']['yaw']}" scope="parent" />
+    <xacro:property name="link6_axis" value="${sec_kinematics['link_6']['axis']}" scope="parent" />
     <!-- Inertia Parameters -->
     <!-- mass -->

Commit message: Add flange and tool0 kinematics properties***
***Update joint origins for flange and tool0

File: urdf/inc/kuka_common.xacro (robot description, xacro)
@@ -186,4 +186,18 @@
     <xacro:property name="link6_yaw" value="${sec_kinematics['link_6']['yaw']}" scope="parent" />
     <xacro:property name="link6_axis" value="${sec_kinematics['link_6']['axis']}" scope="parent" />
+    <!-- Flange -->
+    <xacro:property name="flange_x" value="${sec_kinematics['flange']['x']}" scope="parent" />
+    <xacro:property name="flange_y" value="${sec_kinematics['flange']['y']}" scope="parent" />
+    <xacro:property name="flange_z" value="${sec_kinematics['flange']['z']}" scope="parent" />
+    <xacro:property name="flange_roll" value="${sec_kinematics['flange']['roll']}" scope="parent" />
+    <xacro:property name="flange_pitch" value="${sec_kinematics['flange']['pitch']}" scope="parent" />
+    <xacro:property name="flange_yaw" value="${sec_kinematics['flange']['yaw']}" scope="parent" />
+    <!-- Tool0 -->
+    <xacro:property name="tool0_x" value="${sec_kinematics['tool0']['x']}" scope="parent" />
+    <xacro:property name="tool0_y" value="${sec_kinematics['tool0']['y']}" scope="parent" />
+    <xacro:property name="tool0_z" value="${sec_kinematics['tool0']['z']}" scope="parent" />
+    <xacro:property name="tool0_roll" value="${sec_kinematics['tool0']['roll']}" scope="parent" />
+    <xacro:property name="tool0_pitch" value="${sec_kinematics['tool0']['pitch']}" scope="parent" />
+    <xacro:property name="tool0_yaw" value="${sec_kinematics['tool0']['yaw']}" scope="parent" />
     <!-- Inertia Parameters -->
     <!-- mass -->

File: urdf/kuka_macro.xacro (robot description, xacro)
@@ -263,5 +263,5 @@
       <parent link="${tf_prefix}link_6" />
       <child link="${tf_prefix}flange" />
-      <origin xyz="0 0 0" rpy="0 0 0 " />
+      <origin xyz="0 0 ${flange_z}" rpy="0 ${flange_pitch} 0 " />
     </joint>
     <!-- This frame corresponds to the $TOOL coordinate system in KUKA KRC controllers -->
@@ -270,5 +270,5 @@
       <parent link="${tf_prefix}flange" />
       <child link="${tf_prefix}tool0" />
-      <origin xyz="0 0 0" rpy="0 ${radians(90)} 0" />
+      <origin xyz="0 0 0" rpy="0 ${tool0_pitch} 0" />
     </joint>
   </xacro:macro>

Commit message: Add link axis properties to kuka_common.xacro

File: urdf/inc/kuka_common.xacro (robot description, xacro)
@@ -92,45 +92,51 @@
     <!-- Kinematics -->
     <!-- Link 1 -->
-    <xacro:property name="link1_x" value="${sec_kinematics['link_1']['x']}" scope="parent"/>
-    <xacro:property name="link1_y" value="${sec_kinematics['link_1']['y']}" scope="parent"/>
-    <xacro:property name="link1_z" value="${sec_kinematics['link_1']['z']}" scope="parent"/>
-    <xacro:property name="link1_roll" value="${sec_kinematics['link_1']['roll']}" scope="parent"/>
-    <xacro:property name="link1_pitch" value="${sec_kinematics['link_1']['pitch']}" scope="parent"/>
-    <xacro:property name="link1_yaw" value="${sec_kinematics['link_1']['yaw']}" scope="parent"/>
+    <xacro:property name="link1_x" value="${sec_kinematics['link_1']['x']}" scope="parent" />
+    <xacro:property name="link1_y" value="${sec_kinematics['link_1']['y']}" scope="parent" />
+    <xacro:property name="link1_z" value="${sec_kinematics['link_1']['z']}" scope="parent" />
+    <xacro:property name="link1_roll" value="${sec_kinematics['link_1']['roll']}" scope="parent" />
+    <xacro:property name="link1_pitch" value="${sec_kinematics['link_1']['pitch']}" scope="parent" />
+    <xacro:property name="link1_yaw" value="${sec_kinematics['link_1']['yaw']}" scope="parent" />
+    <xacro:property name="link1_axis" value="${sec_kinematics['link_1']['axis']}" scope="parent" />
     <!-- Link 2 -->
-    <xacro:property name="link2_x" value="${sec_kinematics['link_2']['x']}" scope="parent"/>
-    <xacro:property name="link2_y" value="${sec_kinematics['link_2']['y']}" scope="parent"/>
-    <xacro:property name="link2_z" value="${sec_kinematics['link_2']['z']}" scope="parent"/>
-    <xacro:property name="link2_roll" value="${sec_kinematics['link_2']['roll']}" scope="parent"/>
-    <xacro:property name="link2_pitch" value="${sec_kinematics['link_2']['pitch']}" scope="parent"/>
-    <xacro:property name="link2_yaw" value="${sec_kinematics['link_2']['yaw']}" scope="parent"/>
+    <xacro:property name="link2_x" value="${sec_kinematics['link_2']['x']}" scope="parent" />
+    <xacro:property name="link2_y" value="${sec_kinematics['link_2']['y']}" scope="parent" />
+    <xacro:property name="link2_z" value="${sec_kinematics['link_2']['z']}" scope="parent" />
+    <xacro:property name="link2_roll" value="${sec_kinematics['link_2']['roll']}" scope="parent" />
+    <xacro:property name="link2_pitch" value="${sec_kinematics['link_2']['pitch']}" scope="parent" />
+    <xacro:property name="link2_yaw" value="${sec_kinematics['link_2']['yaw']}" scope="parent" />
+    <xacro:property name="link2_axis" value="${sec_kinematics['link_2']['axis']}" scope="parent" />
     <!-- Link 3 -->
-    <xacro:property name="link3_x" value="${sec_kinematics['link_3']['x']}" scope="parent"/>
-    <xacro:property name="link3_y" value="${sec_kinematics['link_3']['y']}" scope="parent"/>
-    <xacro:property name="link3_z" value="${sec_kinematics['link_3']['z']}" scope="parent"/>
-    <xacro:property name="link3_roll" value="${sec_kinematics['link_3']['roll']}" scope="parent"/>
-    <xacro:property name="link3_pitch" value="${sec_kinematics['link_3']['pitch']}" scope="parent"/>
-    <xacro:property name="link3_yaw" value="${sec_kinematics['link_3']['yaw']}" scope="parent"/>
+    <xacro:property name="link3_x" value="${sec_kinematics['link_3']['x']}" scope="parent" />
+    <xacro:property name="link3_y" value="${sec_kinematics['link_3']['y']}" scope="parent" />
+    <xacro:property name="link3_z" value="${sec_kinematics['link_3']['z']}" scope="parent" />
+    <xacro:property name="link3_roll" value="${sec_kinematics['link_3']['roll']}" scope="parent" />
+    <xacro:property name="link3_pitch" value="${sec_kinematics['link_3']['pitch']}" scope="parent" />
+    <xacro:property name="link3_yaw" value="${sec_kinematics['link_3']['yaw']}" scope="parent" />
+    <xacro:property name="link3_axis" value="${sec_kinematics['link_3']['axis']}" scope="parent" />
     <!-- Link 4 -->
-    <xacro:property name="link4_x" value="${sec_kinematics['link_4']['x']}" scope="parent"/>
-    <xacro:property name="link4_y" value="${sec_kinematics['link_4']['y']}" scope="parent"/>
-    <xacro:property name="link4_z" value="${sec_kinematics['link_4']['z']}" scope="parent"/>
-    <xacro:property name="link4_roll" value="${sec_kinematics['link_4']['roll']}" scope="parent"/>
-    <xacro:property name="link4_pitch" value="${sec_kinematics['link_4']['pitch']}" scope="parent"/>
-    <xacro:property name="link4_yaw" value="${sec_kinematics['link_4']['yaw']}" scope="parent"/>
+    <xacro:property name="link4_x" value="${sec_kinematics['link_4']['x']}" scope="parent" />
+    <xacro:property name="link4_y" value="${sec_kinematics['link_4']['y']}" scope="parent" />
+    <xacro:property name="link4_z" value="${sec_kinematics['link_4']['z']}" scope="parent" />
+    <xacro:property name="link4_roll" value="${sec_kinematics['link_4']['roll']}" scope="parent" />
+    <xacro:property name="link4_pitch" value="${sec_kinematics['link_4']['pitch']}" scope="parent" />
+    <xacro:property name="link4_yaw" value="${sec_kinematics['link_4']['yaw']}" scope="parent" />
+    <xacro:property name="link4_axis" value="${sec_kinematics['link_4']['axis']}" scope="parent" />
     <!-- Link 5 -->
-    <xacro:property name="link5_x" value="${sec_kinematics['link_5']['x']}" scope="parent"/>
-    <xacro:property name="link5_y" value="${sec_kinematics['link_5']['y']}" scope="parent"/>
-    <xacro:property name="link5_z" value="${sec_kinematics['link_5']['z']}" scope="parent"/>
-    <xacro:property name="link5_roll" value="${sec_kinematics['link_5']['roll']}" scope="parent"/>
-    <xacro:property name="link5_pitch" value="${sec_kinematics['link_5']['pitch']}" scope="parent"/>
-    <xacro:property name="link5_yaw" value="${sec_kinematics['link_5']['yaw']}" scope="parent"/>
+    <xacro:property name="link5_x" value="${sec_kinematics['link_5']['x']}" scope="parent" />
+    <xacro:property name="link5_y" value="${sec_kinematics['link_5']['y']}" scope="parent" />
+    <xacro:property name="link5_z" value="${sec_kinematics['link_5']['z']}" scope="parent" />
+    <xacro:property name="link5_roll" value="${sec_kinematics['link_5']['roll']}" scope="parent" />
+    <xacro:property name="link5_pitch" value="${sec_kinematics['link_5']['pitch']}" scope="parent" />
+    <xacro:property name="link5_yaw" value="${sec_kinematics['link_5']['yaw']}" scope="parent" />
+    <xacro:property name="link5_axis" value="${sec_kinematics['link_5']['axis']}" scope="parent" />
     <!-- Link 6 -->
-    <xacro:property name="link6_x" value="${sec_kinematics['link_6']['x']}" scope="parent"/>
-    <xacro:property name="link6_y" value="${sec_kinematics['link_6']['y']}" scope="parent"/>
-    <xacro:property name="link6_z" value="${sec_kinematics['link_6']['z']}" scope="parent"/>
-    <xacro:property name="link6_roll" value="${sec_kinematics['link_6']['roll']}" scope="parent"/>
-    <xacro:property name="link6_pitch" value="${sec_kinematics['link_6']['pitch']}" scope="parent"/>
-    <xacro:property name="link6_yaw" value="${sec_kinematics['link_6']['yaw']}" scope="parent"/>
+    <xacro:property name="link6_x" value="${sec_kinematics['link_6']['x']}" scope="parent" />
+    <xacro:property name="link6_y" value="${sec_kinematics['link_6']['y']}" scope="parent" />
+    <xacro:property name="link6_z" value="${sec_kinematics['link_6']['z']}" scope="parent" />
+    <xacro:property name="link6_roll" value="${sec_kinematics['link_6']['roll']}" scope="parent" />
+    <xacro:property name="link6_pitch" value="${sec_kinematics['link_6']['pitch']}" scope="parent" />
+    <xacro:property name="link6_yaw" value="${sec_kinematics['link_6']['yaw']}" scope="parent" />
+    <xacro:property name="link6_axis" value="${sec_kinematics['link_6']['axis']}" scope="parent" />
     <!-- Inertia Parameters -->
     <!-- mass -->
