Commit message: Add support for 7 dof robot arm in xacros

File: urdf/inc/kuka_common.xacro (robot description, xacro)
@@ -60,5 +60,5 @@
   </xacro:macro>
   <xacro:macro name="read_model_data"
-    params="joint_limits_parameters_file kinematics_parameters_file physical_parameters_file visual_parameters_file force_abs_paths">
+    params="joint_limits_parameters_file kinematics_parameters_file physical_parameters_file visual_parameters_file force_abs_paths dof">
     <xacro:property name="force_abs_paths" value="${force_abs_paths}" scope="parent" />
     <!-- Read .yaml files from disk, load content into properties -->
@@ -137,4 +137,15 @@
     <xacro:property name="joint_6_effort_limit" value="${sec_limits['joint_6']['max_effort']}"
       scope="parent" />
+    <!-- Joint7 -->
+    <xacro:if value="${dof == 7}">
+      <xacro:property name="joint_7_lower_limit" value="${sec_limits['joint_7']['min_position']}"
+        scope="parent" />
+      <xacro:property name="joint_7_upper_limit" value="${sec_limits['joint_7']['max_position']}"
+        scope="parent" />
+      <xacro:property name="joint_7_velocity_limit" value="${sec_limits['joint_7']['max_velocity']}"
+        scope="parent" />
+      <xacro:property name="joint_7_effort_limit" value="${sec_limits['joint_7']['max_effort']}"
+        scope="parent" />
+    </xacro:if>
     <!-- Kinematics -->
     <!-- Link 1 -->
@@ -186,4 +197,14 @@
     <xacro:property name="link6_yaw" value="${sec_kinematics['link_6']['yaw']}" scope="parent" />
     <xacro:property name="link6_axis" value="${sec_kinematics['link_6']['axis']}" scope="parent" />
+    <!-- Link 7 -->
+    <xacro:if value="${dof == 7}">
+      <xacro:property name="link7_x" value="${sec_kinematics['link_7']['x']}" scope="parent" />
+      <xacro:property name="link7_y" value="${sec_kinematics['link_7']['y']}" scope="parent" />
+      <xacro:property name="link7_z" value="${sec_kinematics['link_7']['z']}" scope="parent" />
+      <xacro:property name="link7_roll" value="${sec_kinematics['link_7']['roll']}" scope="parent" />
+      <xacro:property name="link7_pitch" value="${sec_kinematics['link_7']['pitch']}" scope="parent" />
+      <xacro:property name="link7_yaw" value="${sec_kinematics['link_7']['yaw']}" scope="parent" />
+      <xacro:property name="link7_axis" value="${sec_kinematics['link_7']['axis']}" scope="parent" />
+    </xacro:if>
     <!-- Flange -->
     <xacro:property name="flange_x" value="${sec_kinematics['flange']['x']}" scope="parent" />
@@ -216,4 +237,8 @@
     <xacro:property name="link_6_mass" value="${sec_inertia_parameters['link_6_mass']}"
       scope="parent" />
+    <xacro:if value="${dof == 7}">
+      <xacro:property name="link_7_mass" value="${sec_inertia_parameters['link_7_mass']}"
+        scope="parent" />
+    </xacro:if>
     <!-- Link Inertia Parameters -->
     <xacro:property name="intertia_links" value="${sec_inertia_parameters['links']}" scope="parent" />
@@ -246,4 +271,10 @@
     <xacro:property name="link_6_iyy" value="${intertia_links['link_6']['iyy']}" scope="parent" />
     <xacro:property name="link_6_izz" value="${intertia_links['link_6']['izz']}" scope="parent" />
+    <!-- Link 7 -->
+    <xacro:if value="${dof == 7}">
+      <xacro:property name="link_7_ixx" value="${intertia_links['link_7']['ixx']}" scope="parent" />
+      <xacro:property name="link_7_iyy" value="${intertia_links['link_7']['iyy']}" scope="parent" />
+      <xacro:property name="link_7_izz" value="${intertia_links['link_7']['izz']}" scope="parent" />
+    </xacro:if>
   </xacro:macro>
 </robot>

File: urdf/inc/kuka_joint_control.xacro (robot description, xacro)
@@ -5,4 +5,5 @@
     tf_prefix
     initial_positions:=${dict(joint_1=0.0,joint_2=-1.57,joint_3=0.0,joint_4=-1.57,joint_5=0.0,joint_6=0.0)}
+    dof:=6
     ">
     <joint name="${tf_prefix}joint_1">
@@ -42,4 +43,12 @@
       </state_interface>
     </joint>
+    <xacro:if value="${dof == 7}">
+      <joint name="${tf_prefix}joint_7">
+        <command_interface name="position" />
+        <state_interface name="position">
+          <param name="initial_value">0.0</param>
+        </state_interface>
+      </joint>
+    </xacro:if>
   </xacro:macro>
 </robot>

File: urdf/inc/kuka_transmission.xacro (robot description, xacro)
@@ -6,5 +6,5 @@
           this location. Nor can they rely on the existence of the macro.
   -->
-  <xacro:macro name="kuka_arm_transmission" params="tf_prefix">
+  <xacro:macro name="kuka_arm_transmission" params="tf_prefix dof">
     <transmission name="${tf_prefix}joint_1_trans">
       <actuator name="${tf_prefix}joint_1_motor">
@@ -67,4 +67,16 @@
       <type>transmission_interface/SimpleTransmission</type>
     </transmission>
+    <xacro:if value="${dof == 7}">
+      <transmission name="${tf_prefix}joint_7_trans">
+        <actuator name="${tf_prefix}joint_7_motor">
+          <hardwareInterface>EffortJointInterface</hardwareInterface>
+          <mechanicalReduction>1.0</mechanicalReduction>
+        </actuator>
+        <joint name="${tf_prefix}joint_7">
+          <hardwareInterface>hardware_interface/EffortJointInterface</hardwareInterface>
+        </joint>
+        <type>transmission_interface/SimpleTransmission</type>
+      </transmission>
+    </xacro:if>
   </xacro:macro>
 </robot>

File: urdf/kuka.urdf.xacro (robot description, xacro)
@@ -3,8 +3,10 @@
   <!-- robot name parameter -->
   <xacro:arg name="name" default="kuka" />
+  <!-- robot degree of freedom -->
+  <xacro:property name="dof" default="6" />
   <!-- import main macro -->
   <xacro:include filename="$(find kuka_robot_descriptions)/urdf/kuka_macro.xacro" />
   <!-- Possible type are:
-    1.kr6_700_sixx
+    1.kr6_r700_sixx
     2.kr6_r900_sixx
     3.kr10_r1100_2
@@ -49,4 +51,5 @@
     client_port="$(arg client_port)"
     force_abs_paths="$(arg force_abs_paths)"
+    degrees_of_freedom="$(arg dof)"
   >
     <origin xyz="0 0 0" rpy="0 0 0" />          <!-- position robot in the world -->

File: urdf/kuka_macro.xacro (robot description, xacro)
@@ -35,4 +35,5 @@
     visual_parameters_file
     force_abs_paths:=false
+    degrees_of_freedom
     ">
     <xacro:kuka_ros2_control
@@ -42,5 +43,7 @@
       client_port="${client_port}"
       use_fake_hardware="${use_fake_hardware}"
+      dof="${degrees_of_freedom}"
     />
+    <xacro:kuka_arm_transmission tf_prefix="${tf_prefix}" dof="${degrees_of_freedom}" />
     <!-- Load configuration data from the provided .yaml files -->
     <xacro:read_model_data
@@ -49,5 +52,7 @@
       physical_parameters_file="${physical_parameters_file}"
       visual_parameters_file="${visual_parameters_file}"
-      force_abs_paths="${force_abs_paths}" />
+      force_abs_paths="${force_abs_paths}"
+      dof="${degrees_of_freedom}"
+    />
     <!-- Links -main serial chain -->
     <link name="${tf_prefix}base_link">
@@ -184,4 +189,25 @@
       </xacro:inertial_block>
     </link>
+    <!-- Link-7 -->
+    <xacro:if value="${degrees_of_freedom == 7}">
+      <link name="${tf_prefix}link_7">
+        <visual>
+          <origin xyz="0 0 0" rpy="0 0 0" />
+          <geometry>
+            <xacro:get_mesh name="link_7" type="visual" />
+          </geometry>
+          <xacro:get_material name="link_7" type="visual" />
+        </visual>
+        <collision>
+          <geometry>
+            <xacro:get_mesh name="link_7" type="collision" />
+          </geometry>
+        </collision>
+        <xacro:inertial_block mass="${link_7_mass}" ixx="${link_7_ixx}" iyy="${link_7_iyy}"
+          izz="${link_7_izz}">
+          <origin xyz="0 0 0" rpy="0 0 0" />
+        </xacro:inertial_block>
+      </link>
+    </xacro:if>
     <!-- base_joint fixes base_link to the environment -->
     <joint name="${tf_prefix}${parent}-base_link" type="fixed">
@@ -251,4 +277,17 @@
         velocity="${joint_6_velocity_limit}" />
     </joint>
+    <!-- Joint-7 -->
+    <xacro:if value="${degrees_of_freedom == 7}">
+      <joint name="${tf_prefix}joint_7" type="revolute">
+        <parent link="${tf_prefix}link_6" />
+        <child link="${tf_prefix}link_7" />
+        <origin xyz="${link7_x} ${link7_y} ${link7_z}"
+          rpy="${link7_roll} ${link7_pitch} ${link7_yaw}" />
+        <axis xyz="${link7_axis}" />
+        <limit lower="${joint_7_lower_limit}" upper="${joint_7_upper_limit}"
+          effort="${joint_7_effort_limit}"
+          velocity="${joint_7_velocity_limit}" />
+      </joint>
+    </xacro:if>
     <!-- ROS base_link to KUKA $ROBROOT coordinate system transform -->
     <link name="${tf_prefix}base" />
@@ -259,10 +298,20 @@
     </joint>
     <!-- ROS-Industrial 'flange' frame - attachment point for EEF models -->
-    <link name="${tf_prefix}flange" />
-    <joint name="${tf_prefix}joint_6-flange" type="fixed">
-      <parent link="${tf_prefix}link_6" />
-      <child link="${tf_prefix}flange" />
-      <origin xyz="0 0 ${flange_z}" rpy="0 ${flange_pitch} 0 " />
-    </joint>
+    <xacro:if value="${degrees_of_freedom == 7}">
+      <link name="${tf_prefix}flange" />
+      <joint name="${tf_prefix}joint_7-flange" type="fixed">
+        <parent link="${tf_prefix}link_7" />
+        <child link="${tf_prefix}flange" />
+        <origin xyz="0 0 ${flange_z}" rpy="0 ${flange_pitch} 0 " />
+      </joint>
+    </xacro:if>
+    <xacro:if value="${degrees_of_freedom == 6}">
+      <link name="${tf_prefix}flange" />
+      <joint name="${tf_prefix}joint_6-flange" type="fixed">
+        <parent link="${tf_prefix}link_6" />
+        <child link="${tf_prefix}flange" />
+        <origin xyz="0 0 ${flange_z}" rpy="0 ${flange_pitch} 0 " />
+      </joint>
+    </xacro:if>
     <!-- This frame corresponds to the $TOOL coordinate system in KUKA KRC controllers -->
     <link name="${tf_prefix}tool0" />

File: urdf/ros2_control.xacro (robot description, xacro)
@@ -10,4 +10,5 @@
     client_port
     use_fake_hardware
+    dof:=6
     ">
     <ros2_control name="${name}" type="system">
@@ -27,4 +28,5 @@
         tf_prefix="${tf_prefix}"
         initial_positions="${initial_positions}"
+        dof="${dof}"
       />
     </ros2_control>
